Commit message: different model for gazebo to allow first link to be named world

File: urdf/base_example.urdf.xacro (robot description, xacro)
@@ -2,6 +2,6 @@
 <robot name="mobile_base" xmlns:xacro="http://www.ros.org/wiki/xacro">
     <xacro:include filename="$(find gz_virtual_base_system)/urdf/virtual_base_macro.urdf.xacro" />
-    <link name="world"/>
-    <xacro:virtual_base_system world_link="world" base_link="mobile_base_link" />
+    <xacro:arg name="root_link" default="world"/>
+    <xacro:virtual_base_system root_link="$(arg root_link)" base_link="mobile_base_link"/>
     <link name="mobile_base_link">
         <inertial>

File: urdf/virtual_base_macro.urdf.xacro (robot description, xacro)
@@ -5,14 +5,16 @@
     This includes a virtual base link, three joints (x, y, yaw),
     and a ros2_control system interface for controlling the virtual base.
-    @param world_link (String) The unique name of the world link. (parent of the first virtual)
+    @param root_link (String) The unique name of the world link. (parent of the first virtual). Put world for
+    gazebo, odom for ROS2 control.
     @param base_link (String) The unique name of the base link. (child of the last virtual)
   -->
-  <xacro:macro name="virtual_base_system" params="world_link:=world base_link:=base">
+  <xacro:macro name="virtual_base_system" params="root_link:=world base_link:=base">
+  <link name="${root_link}"/>
   <joint name="virtual_joint_x" type="prismatic">
-    <parent link="${world_link}"/>
+    <parent link="${root_link}"/>
     <child link="virtual_base_link_x"/>
     <origin xyz="0 0 0" rpy="0 0 0"/>
     <axis xyz="1 0 0"/>
-    <limit lower="-1000" upper="1000" effort="1000" velocity="1"/>
+    <limit lower="-100000" upper="100000" effort="100000" velocity="1"/>
   </joint>
   <joint name="virtual_joint_y" type="prismatic">
@@ -21,5 +23,5 @@
     <origin xyz="0 0 0" rpy="0 0 0"/>
     <axis xyz="0 1 0"/>
-    <limit lower="-1000" upper="1000" effort="1000" velocity="1"/>
+    <limit lower="-100000" upper="100000" effort="100000" velocity="1"/>
   </joint>
   <joint name="virtual_joint_yaw" type="continuous">
@@ -30,5 +32,4 @@
   </joint>
   <link name="virtual_base_link_x">
-    <origin xyz="0 0 0.0" rpy="0 0 0"/>
     <inertial>
       <origin xyz="0 0 0" rpy="0 0 0"/>
@@ -38,5 +39,4 @@
   </link>
   <link name="virtual_base_link_y">
-    <origin xyz="0 0 0" rpy="0 0 0"/>
     <inertial>
       <origin xyz="0 0 0" rpy="0 0 0"/>
